File: board/board.kicad_pcb (KiCad board)
At the start: 2 copper layers, 21 x 13 mm, 1 part

Commit message: initial
Parts:
- added C1: 100nF, Capacitor_SMD:C_0603_1608Metric, F.Cu at (143.0, 112.0)
- added J1: 007_ADC, on_edge:on_edge_2x05_device, F.Cu at (140.0, 96.5)
- added J2: 011_GPIO, on_edge:on_edge_2x05_device, F.Cu at (140.0, 144.5)
- added J3: 007_ADC, on_edge:on_edge_2x05_host, F.Cu at (161.0, 96.5)
- added J4: 007_ADC, on_edge:on_edge_2x05_host, F.Cu at (161.0, 112.5)
- added J5: 007_ADC, on_edge:on_edge_2x05_host, F.Cu at (161.0, 128.5)
- added J6: 007_ADC, on_edge:on_edge_2x05_host, F.Cu at (161.0, 144.5)
- added U1: Val**, b109:ADG707BRUZ-REEL7, F.Cu at (149.0, 112.0)
- moved LOGO1 44.3 mm to (150.4, 143.2)
Routing:
- net GND: track 0.00 -> 145.9 mm, vias 0 -> 9
- net /mux/EN: track 0.00 -> 114.3 mm, vias 0 -> 7
- net Net-(J1-Pad10): track 0.00 -> 95.1 mm, vias 0 -> 6
- net /mux/S7B: track 0.00 -> 43.7 mm, vias 0 -> 2
- net /mux/S8A: track 0.00 -> 40.0 mm, vias 0 -> 2
- net /mux/S7A: track 0.00 -> 36.9 mm, vias 0 -> 2
- net /mux/S8B: track 0.00 -> 35.5 mm, vias 0 -> 1
- net /mux/A2: track 0.00 -> 35.0 mm, vias 0 -> 2
- net /mux/A1: track 0.00 -> 33.8 mm, vias 0 -> 2
- net /mux/A0: track 0.00 -> 32.3 mm, vias 0 -> 2
- net /mux/DA: track 0.00 -> 28.3 mm, vias 0 -> 2
- net /mux/S5B: track 0.00 -> 26.3 mm, vias 0 -> 2
- net /mux/S1A: track 0.00 -> 26.1 mm, vias 0 -> 2
- net /mux/S6A: track 0.00 -> 24.3 mm, vias 0 -> 2
- net /mux/S2A: track 0.00 -> 23.8 mm, vias 0 -> 2
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Other:
- board size 21 x 13 mm -> 21 x 61 mm
- board text added: "osf.007"
- board text added: "osf.011"
- board text added: "osf.b0109.v1.0"
