File: board/board.kicad_pcb (KiCad board)
At the start: 2 copper layers, 21 x 61 mm, 9 parts, among them J1 007_ADC, J2 011_GPIO, J3 007_ADC, J4 007_ADC, J5 007_ADC, J6 007_ADC, U1 Val**

Commit message: added lcsc part numbers
Parts:
- U1: value Val** -> ADG707BRUZ-REEL7
