File: board/board.kicad_sch (KiCad schematic)
At the start: 7 parts, among them J1 007_ADC, J2 011_GPIO, J3 007_ADC, J4 007_ADC, J5 007_ADC, J6 007_ADC

Commit message: added lcsc part numbers
Parts:
- J1: lcsc (none) -> C14663
